File: ra5_2022.kicad_pcb (KiCad board)
At the start: 2 copper layers, 16 parts, among them CN1 KF250-3.5-2P-2, Q1 Q_PMOS_GSD, U1 AP63203WU, U2 B0303S-1W_C883455

Commit message: Add MCU and M90E32AS sheets, import connector/switch/MCU parts
Adds the mcu.kicad_sch and m90e32as.kicad_sch hierarchical sheets and
wires them into the root schematic and PCB. Imports several LCSC parts
into the project-local ra5_2022 library (symbols/footprints/3D models):
USB-C connectors, TQFP-48 MCU footprint, tactile switch, and the
DB126V-5.0-2P terminal block, plus adds schematic-only symbols for the
MX15EDGRHC-3.5-2x03P receptacle and its MX15EDGKNH-3.5-2x03P mating
plug (BOM-only, not placed on board). Checks in CLAUDE.md.
Parts:
- added C10: 100nF, Capacitor_SMD:C_0402_1005Metric, F.Cu at (210.7, 79.0)
- added C11: 22uF, Capacitor_SMD:C_0402_1005Metric, F.Cu at (210.7, 81.0)
- added C12: 100nF, Capacitor_SMD:C_0402_1005Metric, F.Cu at (210.7, 82.9)
- added C13: 100nF, Capacitor_SMD:C_0402_1005Metric, F.Cu at (210.7, 84.9)
- added C14: 100nF, Capacitor_SMD:C_0402_1005Metric, F.Cu at (205.8, 83.5)
- added C15: 10uF, Capacitor_SMD:C_0603_1608Metric, F.Cu at (200.8, 92.7)
- added C16: 100nF, Capacitor_SMD:C_0402_1005Metric, F.Cu at (205.8, 85.4)
- added C17: 100nF, Capacitor_SMD:C_0402_1005Metric, F.Cu at (205.8, 87.4)
- added C18: 100nF, Capacitor_SMD:C_0402_1005Metric, F.Cu at (205.8, 89.4)
- added C19: 33nF, Capacitor_SMD:C_0402_1005Metric, F.Cu at (271.3, 65.9)
- added C20: 33nF, Capacitor_SMD:C_0402_1005Metric, F.Cu at (271.3, 67.9)
- added C21: 33nF, Capacitor_SMD:C_0402_1005Metric, F.Cu at (274.1, 62.0)
- added C22: 33nF, Capacitor_SMD:C_0402_1005Metric, F.Cu at (274.1, 64.0)
- added C23: 33nF, Capacitor_SMD:C_0402_1005Metric, F.Cu at (274.1, 65.9)
- added C24: 33nF, Capacitor_SMD:C_0402_1005Metric, F.Cu at (274.1, 67.9)
- added C25: 33nF, Capacitor_SMD:C_0402_1005Metric, F.Cu at (277.0, 62.0)
- added C26: 33nF, Capacitor_SMD:C_0402_1005Metric, F.Cu at (277.0, 64.0)
- added C27: 33nF, Capacitor_SMD:C_0402_1005Metric, F.Cu at (277.0, 65.9)
- added C28: 33nF, Capacitor_SMD:C_0402_1005Metric, F.Cu at (277.0, 67.9)
- added C29: 100nF, Capacitor_SMD:C_0402_1005Metric, F.Cu at (116.0, 140.0)
- added C5: 4.7uF, Capacitor_SMD:C_0402_1005Metric, F.Cu at (205.8, 81.5)
- added C6: 33nF, Capacitor_SMD:C_0402_1005Metric, F.Cu at (271.3, 62.0)
- added C7: 33nF, Capacitor_SMD:C_0402_1005Metric, F.Cu at (271.3, 64.0)
- added C8: 10uF, Capacitor_SMD:C_0603_1608Metric, F.Cu at (232.2, 128.8)
- added C9: 10uF, Capacitor_SMD:C_0603_1608Metric, F.Cu at (214.1, 79.3)
- added D4: PESD5V0L4UF, Package_TO_SOT_SMD:SOT-886, F.Cu at (236.4, 119.6)
- added D5: D_Schottky, Diode_SMD:D_SOD-123, F.Cu at (228.1, 127.9)
- added D6: LED, LED_SMD:LED_0603_1608Metric, F.Cu at (271.9, 70.2)
- added D7: LED, LED_SMD:LED_0603_1608Metric, F.Cu at (271.9, 72.8)
- added D8: LED, LED_SMD:LED_0603_1608Metric, F.Cu at (271.9, 75.4)
- added J1: USB_C_Receptacle, Connector_USB:USB_C_Receptacle_GCT_USB4115-03-C, F.Cu at (139.8, 107.7)
- added J2: MX15EDGRHC-3.5-2x03P, ra5_2022:CONN-TH_6P-P3.50x2.50_MAX_MX15EDGRHC-3.5-2x03P, F.Cu at (184.8, 102.1)
- added R10: 80R, Resistor_SMD:R_0603_1608Metric, F.Cu at (267.8, 62.3)
- added R11: 80R, Resistor_SMD:R_0603_1608Metric, F.Cu at (267.8, 64.8)
- added R12: 80R, Resistor_SMD:R_0603_1608Metric, F.Cu at (267.8, 67.3)
- added R13: 12M, Resistor_SMD:R_1206_3216Metric, F.Cu at (251.8, 62.7)
- added R14: 12M, Resistor_SMD:R_1206_3216Metric, F.Cu at (251.8, 66.0)
- added R15: 12M, Resistor_SMD:R_1206_3216Metric, F.Cu at (251.8, 69.3)
- added R16: 12M, Resistor_SMD:R_1206_3216Metric, F.Cu at (251.8, 72.6)
- added R17: 12M, Resistor_SMD:R_1206_3216Metric, F.Cu at (251.8, 75.9)
- added R18: 12M, Resistor_SMD:R_1206_3216Metric, F.Cu at (251.8, 79.2)
- added R19: 12M, Resistor_SMD:R_1206_3216Metric, F.Cu at (251.8, 82.5)
- added R20: 1k, Resistor_SMD:R_0402_1005Metric, F.Cu at (267.3, 84.6)
- added R21: 1k, Resistor_SMD:R_0402_1005Metric, F.Cu at (267.3, 86.6)
- added R22: 12M, Resistor_SMD:R_1206_3216Metric, F.Cu at (257.4, 62.7)
- added R23: 12M, Resistor_SMD:R_1206_3216Metric, F.Cu at (257.4, 66.0)
- added R24: 12M, Resistor_SMD:R_1206_3216Metric, F.Cu at (257.4, 69.3)
- added R25: 12M, Resistor_SMD:R_1206_3216Metric, F.Cu at (257.4, 72.6)
- added R26: 12M, Resistor_SMD:R_1206_3216Metric, F.Cu at (257.4, 75.9)
- added R27: 12M, Resistor_SMD:R_1206_3216Metric, F.Cu at (257.4, 79.2)
- added R28: 12M, Resistor_SMD:R_1206_3216Metric, F.Cu at (257.4, 82.5)
- added R29: 1k, Resistor_SMD:R_0402_1005Metric, F.Cu at (267.3, 88.6)
- added R30: 1k, Resistor_SMD:R_0402_1005Metric, F.Cu at (267.3, 90.6)
- added R31: 12M, Resistor_SMD:R_1206_3216Metric, F.Cu at (263.0, 62.7)
- added R32: 12M, Resistor_SMD:R_1206_3216Metric, F.Cu at (263.0, 66.0)
- added R33: 12M, Resistor_SMD:R_1206_3216Metric, F.Cu at (263.0, 69.3)
- added R34: 12M, Resistor_SMD:R_1206_3216Metric, F.Cu at (263.0, 72.6)
- added R35: 12M, Resistor_SMD:R_1206_3216Metric, F.Cu at (263.0, 75.9)
- added R36: 12M, Resistor_SMD:R_1206_3216Metric, F.Cu at (263.0, 79.2)
- added R37: 12M, Resistor_SMD:R_1206_3216Metric, F.Cu at (263.0, 82.5)
- added R38: 1k, Resistor_SMD:R_0402_1005Metric, F.Cu at (270.2, 84.6)
- added R39: 1k, Resistor_SMD:R_0402_1005Metric, F.Cu at (270.2, 86.6)
- added R40: 1k, Resistor_SMD:R_0402_1005Metric, F.Cu at (270.2, 88.6)
- added R41: 2.4R, Resistor_SMD:R_0603_1608Metric, F.Cu at (267.8, 69.8)
- added R42: 2.4R, Resistor_SMD:R_0603_1608Metric, F.Cu at (267.8, 72.3)
- added R43: 1k, Resistor_SMD:R_0402_1005Metric, F.Cu at (270.2, 90.6)
- added R44: 2.4R, Resistor_SMD:R_0603_1608Metric, F.Cu at (267.8, 74.8)
- added R45: 2.4R, Resistor_SMD:R_0603_1608Metric, F.Cu at (267.8, 77.3)
- added R46: 1k, Resistor_SMD:R_0402_1005Metric, F.Cu at (273.1, 84.6)
- added R47: 1k, Resistor_SMD:R_0402_1005Metric, F.Cu at (273.1, 86.6)
- added R48: 2.4R, Resistor_SMD:R_0603_1608Metric, F.Cu at (267.8, 79.8)
- added R49: 2.4R, Resistor_SMD:R_0603_1608Metric, F.Cu at (267.8, 82.3)
- added R5: 5.1k, Resistor_SMD:R_0603_1608Metric, F.Cu at (223.2, 119.2)
- added R50: 1k, Resistor_SMD:R_0402_1005Metric, F.Cu at (273.1, 88.6)
- added R51: 1k, Resistor_SMD:R_0402_1005Metric, F.Cu at (273.1, 90.6)
- added R52: 10k, Resistor_SMD:R_0402_1005Metric, F.Cu at (116.0, 134.1)
- added R53: 430R, Resistor_SMD:R_0402_1005Metric, F.Cu at (163.0, 97.5)
- added R54: 560R, Resistor_SMD:R_0402_1005Metric, F.Cu at (116.0, 138.1)
- added R55: 430R, Resistor_SMD:R_0402_1005Metric, F.Cu at (254.5, 110.0)
- added R56: 560R, Resistor_SMD:R_0402_1005Metric, F.Cu at (254.5, 112.0)
- added R57: 270R, Resistor_SMD:R_0402_1005Metric, F.Cu at (254.5, 114.0)
- added R58: 560R, Resistor_SMD:R_0402_1005Metric, F.Cu at (254.5, 116.0)
- added R59: 430R, Resistor_SMD:R_0402_1005Metric, F.Cu at (254.5, 118.0)
- added R6: 5.1k, Resistor_SMD:R_0603_1608Metric, F.Cu at (223.2, 121.7)
- added R60: 560R, Resistor_SMD:R_0402_1005Metric, F.Cu at (254.5, 119.9)
- added R61: 430R, Resistor_SMD:R_0402_1005Metric, F.Cu at (208.0, 45.0)
- added R62: 560R, Resistor_SMD:R_0402_1005Metric, F.Cu at (208.0, 47.0)
- added R63: 430R, Resistor_SMD:R_0402_1005Metric, F.Cu at (208.0, 49.0)
- added R64: 560R, Resistor_SMD:R_0402_1005Metric, F.Cu at (208.0, 51.0)
- added R65: 430R, Resistor_SMD:R_0402_1005Metric, F.Cu at (208.0, 53.0)
- added R66: 560R, Resistor_SMD:R_0402_1005Metric, F.Cu at (208.0, 54.9)
- added R67: 430R, Resistor_SMD:R_0402_1005Metric, F.Cu at (208.0, 56.9)
- added R68: 560R, Resistor_SMD:R_0402_1005Metric, F.Cu at (208.0, 58.9)
- added R7: 10k, Resistor_SMD:R_0402_1005Metric, F.Cu at (223.2, 124.2)
- added R8: 10k, Resistor_SMD:R_0402_1005Metric, F.Cu at (213.6, 81.5)
- added R9: 10k, Resistor_SMD:R_0402_1005Metric, F.Cu at (213.6, 83.5)
- added SW1: SW_Push, Button_Switch_SMD:SW_SPST_TL3342, F.Cu at (124.0, 101.5)
- added SW2: SW_Push, Button_Switch_SMD:SW_SPST_TL3342, F.Cu at (124.0, 108.5)
- added U10: DB126V-5.0-2P-BK-P, ra5_2022:CONN-TH_2P-P5.00_DIBO_DB126V-5.0-2P-BU-P, F.Cu at (185.0, 88.5)
- added U3: ESP32-C6-MINI-1, RF_Module:ESP32-C6-MINI-1, F.Cu at (169.4, 107.5)
- added U4: AMS1117-3.3, Package_TO_SOT_SMD:SOT-223-3_TabPin2, F.Cu at (230.1, 122.1)
- added U5: ATM90E32AS-AU-R, ra5_2022:TQFP-48_L7.0-W7.0-P0.50-LS9.0-BL, F.Cu at (198.9, 86.0)
- added U6: K3-2268P, ra5_2022:SW-SMD_12P-L14.9-W4.9_K3-2268P, F.Cu at (257.1, 88.7)
- added U7: TLP291-4, Package_SO:SOIC-16_4.55x10.3mm_P1.27mm, F.Cu at (109.8, 139.1)
- added U8: TLP291-4, Package_SO:SOIC-16_4.55x10.3mm_P1.27mm, F.Cu at (214.2, 50.0)
- added U9: DB126V-5.0-2P-BK-P, ra5_2022:CONN-TH_2P-P5.00_DIBO_DB126V-5.0-2P-BU-P, F.Cu at (185.0, 78.5)
- added Y1: ABM8G-16.384MHZ-18-D2Y-T, Crystal:Crystal_SMD_3225-4Pin_3.2x2.5mm, F.Cu at (192.1, 92.3)
- Q1: value Q_PMOS_GSD -> PJM2309PSC
Connections:
- U2 pad 3: unconnected-(U2--VO-Pad3) -> GND2
- U2 pad 4: unconnected-(U2-+VO-Pad4) -> VDD2
