File: mcu.kicad_sch (KiCad schematic)
At the start: 24 parts, among them J1 Bus_M.2_Socket_E, J2 Conn_01x04_Socket, U1 STM8S003F3P, U5 ISO7741N1-Y, U6 CS817X20LS, U7 AMS1117-3.3

Commit message: Fix USB_90R/HighSpeed netclass clearance for M.2 socket pitch, route USB diff pair, add board render doc
Netclass clearance (0.25mm) exceeded the J1 M.2 socket's actual 0.5mm-pitch
pad spacing (~0.2mm) and the USB_90R diff pair gap (0.1mm), blocking the
interactive router from escaping J1's pads. Lowered USB_90R and HighSpeed
clearance to 0.2mm and the board's global min_clearance/min_connection to
match, plus a custom rule permitting the 0.1mm DP/DN internal gap. Routed
the USB_DP/USB_DN differential pair from J1 to D3.

Added view/ with finished-board renders and a short board description.
Parts:
- removed D3: PESD5V0L2UM,315, ra5_2022:SOT-883-3_L1.0-W0.6-BR, symbol ra5_2022:PESD5V0L2UM,315
- added D3: USBLC6-2SC6, ra5_2022:SOT-23-6_L2.9-W1.6-P0.95-LS2.8-BL, symbol ra5_2022:USBLC6-2SC6
Connections:
- net +5V_USB: now also D3.5
- net Digital IO/DIN1_MCU: now also U1.15 (PC5); no longer U1.13 (PC3)
- net Digital IO/DIN2_MCU: now also U1.16 (PC6); no longer U1.14 (PC4)
- net Digital IO/DO1_MCU: now also U1.14 (PC4); no longer U1.15 (PC5)
- net Digital IO/DO2_MCU: now also U1.13 (PC3); no longer U1.16 (PC6)
- net GND: now also D3.2
- net USB_DN: now also D3.4; no longer USB1.A7 (DN1), USB1.B7 (DN2)
- net USB_DP: now also D3.6; no longer USB1.A6 (DP1), USB1.B6 (DP2)
- new net USB_D+: D3.1, USB1.A6 (DP1), USB1.B6 (DP2)
- new net USB_D-: D3.3, USB1.A7 (DN1), USB1.B7 (DN2)
